File: hardware/al8843/al8843.kicad_pcb (KiCad board)
At the start: 2 copper layers, 18 parts, among them J3 LED_A, J4 LED_K, U1 AL8843

Commit message: update to latest kicad
Other:
- board outline added: 42.1 x 24.2 mm
- net class Default removed
