File: hardware/al8843/al8843.sch (KiCad schematic (older format))
At the start: 18 parts, among them J1 Conn_01x02, J2 Conn_01x02, J3 LED_A, J4 LED_K, U1 AL8843

Commit message: clean-up
Connections:
- wire segments 63 -> 57
Other:
- moved on the sheet: C1, C2, C3, C4, C5, C6, D1, J1, J2, J3, J4, L1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
